Commit message: Phase 4 final: fix Gazebo friction, adjust demo waypoints and loops

File: src/amr_sim/urdf/macros.xacro (robot description, xacro)
@@ -25,6 +25,17 @@
                 <xacro:sphere_inertia m="${trolley_wheel_mass}" r="${trolley_wheel_radius}"/>
             </inertial>
-            <mu>0.0</mu>
         </link>
+        <gazebo reference="${cardinality}_${dexterity}_wheel">
+            <collision>
+                <surface>
+                    <friction>
+                        <ode>
+                            <mu>0.0</mu>
+                            <mu2>0.0</mu2>
+                        </ode>
+                    </friction>
+                </surface>
+            </collision>
+        </gazebo>
         <joint name="${cardinality}_${dexterity}_wheel_joint" type="fixed">
             <parent link="base_link"/>
@@ -51,6 +62,17 @@
                 <xacro:cylinder_inertia m="${traction_wheel_mass}" r="${traction_wheel_radius}" h="${traction_wheel_width}"/>
             </inertial>
-            <mu>5.0</mu>
         </link>
+        <gazebo reference="${cardinality}_${dexterity}_wheel">
+            <collision>
+                <surface>
+                    <friction>
+                        <ode>
+                            <mu>5.0</mu>
+                            <mu2>5.0</mu2>
+                        </ode>
+                    </friction>
+                </surface>
+            </collision>
+        </gazebo>
         <joint name="${cardinality}_${dexterity}_wheel_joint" type="continuous">
             <parent link="base_link"/>
