Commit message: feat(fleet): optimize multi-robot tf tree, vectorized map fusion, and navigation stability
- Add tf_relay node to bridge per-robot tf/tf_static to global tree
- Migrate SLAM, Nav2, and readiness coordinators to base_footprint
- Vectorize map_fusion_node with NumPy for fast, bounded occupancy grid merges
- Improve mission_manager_node concurrency with MultiThreadedExecutor
- Add Gazebo resource path environment variables to launch files
- Update URDF mesh URIs to package:// schema
- Ignore ROS 2 bag files in .gitignore

File: src/amr_sim/urdf/bcr_bot_amr1.xacro (robot description, xacro)
@@ -28,4 +28,5 @@
     <xacro:property name="camera_height" value="0.10"/>
     <xacro:property name="camera_horizontal_fov" value="60"/>
+    <xacro:arg name="robot_name" default="bcr_bot_amr1"/>
     <xacro:arg name="robot_namespace" default=""/>
     <xacro:arg name="wheel_odom_topic" default="odom" />
@@ -71,5 +72,5 @@
             <origin xyz="0 0 -0.205" rpy="0 0 0" />
             <geometry>
-                <mesh filename="file://$(find amr_sim)/meshes/bcr_bot_mesh.dae" scale="1 1 1"/>
+                <mesh filename="package://amr_sim/meshes/bcr_bot_mesh.dae" scale="1 1 1"/>
             </geometry>
         </visual>
@@ -142,5 +143,5 @@
                 <origin xyz="0 0 0" rpy="0 0 0" />
                 <geometry>
-                    <mesh filename="file://$(find amr_sim)/meshes/kinect/d415.dae"/>
+                    <mesh filename="package://amr_sim/meshes/kinect/d415.dae"/>
                 </geometry>
                 <material name="black"/>
@@ -176,5 +177,5 @@
                 <origin xyz="0 0 0" rpy="0 0 0" />
                 <geometry>
-                    <mesh filename="file://$(find amr_sim)/meshes/kinect/d415.dae"/>
+                    <mesh filename="package://amr_sim/meshes/kinect/d415.dae"/>
                 </geometry>
                 <material name="black"/>

File: src/amr_sim/urdf/bcr_bot_amr2.xacro (robot description, xacro)
@@ -29,4 +29,5 @@
     <xacro:property name="camera_height" value="0.10"/>
     <xacro:property name="camera_horizontal_fov" value="60"/>
+    <xacro:arg name="robot_name" default="bcr_bot_amr2"/>
     <xacro:arg name="robot_namespace" default=""/>
     <xacro:arg name="wheel_odom_topic" default="odom" />
@@ -72,5 +73,5 @@
             <origin xyz="0 0 -0.205" rpy="0 0 0" />
             <geometry>
-                <mesh filename="file://$(find amr_sim)/meshes/bcr_bot_mesh.dae" scale="0.9 0.9 0.9"/>
+                <mesh filename="package://amr_sim/meshes/bcr_bot_mesh.dae" scale="0.9 0.9 0.9"/>
             </geometry>
         </visual>
@@ -143,5 +144,5 @@
                 <origin xyz="0 0 0" rpy="0 0 0" />
                 <geometry>
-                    <mesh filename="file://$(find amr_sim)/meshes/kinect/d415.dae"/>
+                    <mesh filename="package://amr_sim/meshes/kinect/d415.dae"/>
                 </geometry>
                 <material name="black"/>
@@ -177,5 +178,5 @@
                 <origin xyz="0 0 0" rpy="0 0 0" />
                 <geometry>
-                    <mesh filename="file://$(find amr_sim)/meshes/kinect/d415.dae"/>
+                    <mesh filename="package://amr_sim/meshes/kinect/d415.dae"/>
                 </geometry>
                 <material name="black"/>

File: src/amr_sim/urdf/gz.xacro (robot description, xacro)
@@ -21,27 +21,10 @@
             <min_angular_acceleration>-1.0</min_angular_acceleration>
             <topic>/bcr_bot_amr1/cmd_vel</topic>
-            <xacro:if value="${odometry_source == 'encoders'}">
-                <odom_topic>$(arg wheel_odom_topic)</odom_topic>
-                <tf_topic>/tf</tf_topic>
-            </xacro:if>
+            <odom_topic>$(arg wheel_odom_topic)</odom_topic>
+            <tf_topic>/model/$(arg robot_name)/tf</tf_topic>
             <frame_id>$(arg robot_name)/odom</frame_id>
             <child_frame_id>$(arg robot_name)/base_footprint</child_frame_id>
         </plugin>
     </gazebo>
-    <!-- ............................. ground truth .................................... -->
-    <xacro:if value="${odometry_source == 'world'}">
-    <gazebo>
-        <plugin filename="libgz-sim-odometry-publisher-system"
-            name="gz::sim::systems::OdometryPublisher">
-            <odom_frame>$(arg robot_name)/odom</odom_frame>
-            <robot_base_frame>$(arg robot_name)/base_footprint</robot_base_frame>
-            <odom_topic>$(arg wheel_odom_topic)</odom_topic>
-            <tf_topic>/tf</tf_topic>
-            <dimensions>2</dimensions>
-            <!-- Match the 30 Hz lidar so scan-time TF interpolation stays current. -->
-            <odom_publish_frequency>30</odom_publish_frequency>
-        </plugin>
-    </gazebo>
-    </xacro:if>
     <!-- ........................... 2D LIDAR config ................................... -->
     <xacro:if value="$(arg two_d_lidar_enabled)">

File: src/amr_sim/urdf/gz_amr2.xacro (robot description, xacro)
@@ -22,27 +22,10 @@
             <min_angular_acceleration>-2.5</min_angular_acceleration>
             <topic>/bcr_bot_amr2/cmd_vel</topic>
-            <xacro:if value="${odometry_source == 'encoders'}">
-                <odom_topic>$(arg wheel_odom_topic)</odom_topic>
-                <tf_topic>/tf</tf_topic>
-            </xacro:if>
+            <odom_topic>$(arg wheel_odom_topic)</odom_topic>
+            <tf_topic>/model/$(arg robot_name)/tf</tf_topic>
             <frame_id>$(arg robot_name)/odom</frame_id>
             <child_frame_id>$(arg robot_name)/base_footprint</child_frame_id>
         </plugin>
     </gazebo>
-    <!-- ............................. ground truth .................................... -->
-    <xacro:if value="${odometry_source == 'world'}">
-    <gazebo>
-        <plugin filename="libgz-sim-odometry-publisher-system"
-            name="gz::sim::systems::OdometryPublisher">
-            <odom_frame>$(arg robot_name)/odom</odom_frame>
-            <robot_base_frame>$(arg robot_name)/base_footprint</robot_base_frame>
-            <odom_topic>$(arg wheel_odom_topic)</odom_topic>
-            <tf_topic>/tf</tf_topic>
-            <dimensions>2</dimensions>
-            <!-- Match the 30 Hz lidar so scan-time TF interpolation stays current. -->
-            <odom_publish_frequency>30</odom_publish_frequency>
-        </plugin>
-    </gazebo>
-    </xacro:if>
     <!-- ........................... 2D LIDAR config ................................... -->
     <xacro:if value="$(arg two_d_lidar_enabled)">

Commit message: fix(sim, bsp): enhance ramp climbing friction, wheel contact mechanics, and TF ground filtering

File: src/amr_sim/urdf/bcr_bot_amr1.xacro (robot description, xacro)
@@ -14,6 +14,6 @@
     <xacro:property name="trolley_wheel_friction" value="0.0"/>
     <xacro:property name="trolley_wheel_radius" value="0.06"/>
-    <!-- a small constant -->
-    <xacro:property name="eps" value="0.002"/>
+    <!-- a small constant for drive wheel ground engagement -->
+    <xacro:property name="eps" value="0.008"/>
     <xacro:property name="traction_wheel_radius" value="0.1"/>
     <xacro:property name="traction_wheel_width" value="0.05"/>

File: src/amr_sim/urdf/bcr_bot_amr2.xacro (robot description, xacro)
@@ -15,6 +15,6 @@
     <xacro:property name="trolley_wheel_friction" value="0.0"/>
     <xacro:property name="trolley_wheel_radius" value="0.06"/>
-    <!-- a small constant -->
-    <xacro:property name="eps" value="0.002"/>
+    <!-- a small constant for drive wheel ground engagement -->
+    <xacro:property name="eps" value="0.008"/>
     <xacro:property name="traction_wheel_radius" value="0.1"/>
     <xacro:property name="traction_wheel_width" value="0.05"/>

File: src/amr_sim/urdf/gz.xacro (robot description, xacro)
@@ -16,8 +16,8 @@
             <max_linear_velocity>1.0</max_linear_velocity>
             <max_angular_velocity>1.0</max_angular_velocity>
-            <max_linear_acceleration>1.0</max_linear_acceleration>
-            <max_angular_acceleration>1.0</max_angular_acceleration>
-            <min_linear_acceleration>-1.0</min_linear_acceleration>
-            <min_angular_acceleration>-1.0</min_angular_acceleration>
+            <max_linear_acceleration>2.5</max_linear_acceleration>
+            <max_angular_acceleration>2.5</max_angular_acceleration>
+            <min_linear_acceleration>-2.5</min_linear_acceleration>
+            <min_angular_acceleration>-2.5</min_angular_acceleration>
             <topic>/bcr_bot_amr1/cmd_vel</topic>
             <odom_topic>$(arg wheel_odom_topic)</odom_topic>

File: src/amr_sim/urdf/macros.xacro (robot description, xacro)
@@ -33,6 +33,15 @@
                             <mu>0.0</mu>
                             <mu2>0.0</mu2>
+                            <slip1>1.0</slip1>
+                            <slip2>1.0</slip2>
                         </ode>
                     </friction>
+                    <contact>
+                        <ode>
+                            <kp>100000.0</kp>
+                            <kd>10.0</kd>
+                            <min_depth>0.015</min_depth>
+                        </ode>
+                    </contact>
                 </surface>
             </collision>
@@ -68,8 +77,17 @@
                     <friction>
                         <ode>
-                            <mu>5.0</mu>
-                            <mu2>5.0</mu2>
+                            <mu>10.0</mu>
+                            <mu2>10.0</mu2>
+                            <slip1>0.0</slip1>
+                            <slip2>0.0</slip2>
                         </ode>
                     </friction>
+                    <contact>
+                        <ode>
+                            <kp>10000000.0</kp>
+                            <kd>1.0</kd>
+                            <min_depth>0.001</min_depth>
+                        </ode>
+                    </contact>
                 </surface>
             </collision>

Commit message: fix(physics, nav2): ensure drive wheel traction on 10deg ramp transition and tune inflation potential for narrow ramp clearance

File: src/amr_sim/urdf/bcr_bot_amr1.xacro (robot description, xacro)
@@ -15,5 +15,5 @@
     <xacro:property name="trolley_wheel_radius" value="0.06"/>
     <!-- a small constant for drive wheel ground engagement -->
-    <xacro:property name="eps" value="0.008"/>
+    <xacro:property name="eps" value="0.022"/>
     <xacro:property name="traction_wheel_radius" value="0.1"/>
     <xacro:property name="traction_wheel_width" value="0.05"/>

File: src/amr_sim/urdf/bcr_bot_amr2.xacro (robot description, xacro)
@@ -16,5 +16,5 @@
     <xacro:property name="trolley_wheel_radius" value="0.06"/>
     <!-- a small constant for drive wheel ground engagement -->
-    <xacro:property name="eps" value="0.008"/>
+    <xacro:property name="eps" value="0.022"/>
     <xacro:property name="traction_wheel_radius" value="0.1"/>
     <xacro:property name="traction_wheel_width" value="0.05"/>

File: src/amr_sim/urdf/macros.xacro (robot description, xacro)
@@ -39,7 +39,7 @@
                     <contact>
                         <ode>
-                            <kp>100000.0</kp>
-                            <kd>10.0</kd>
-                            <min_depth>0.015</min_depth>
+                            <kp>50000.0</kp>
+                            <kd>100.0</kd>
+                            <min_depth>0.035</min_depth>
                         </ode>
                     </contact>

Commit message: fix(physics, bsp, slam, mission): raise chassis collision clearance, fix ramp ground filter boundaries, restore continuous slam registration, and implement conflict yielding coordinator

File: src/amr_sim/urdf/bcr_bot_amr1.xacro (robot description, xacro)
@@ -64,5 +64,5 @@
     <link name="chassis_link">
         <collision>
-            <origin xyz="0 0 -0.05" rpy="0 0 0" />
+            <origin xyz="0 0 0.0" rpy="0 0 0" />
             <geometry>
                 <box size="${chassis_length} ${chassis_width} ${chassis_height}"/>

File: src/amr_sim/urdf/bcr_bot_amr2.xacro (robot description, xacro)
@@ -65,5 +65,5 @@
     <link name="chassis_link">
         <collision>
-            <origin xyz="0 0 -0.05" rpy="0 0 0" />
+            <origin xyz="0 0 0.0" rpy="0 0 0" />
             <geometry>
                 <box size="${chassis_length} ${chassis_width} ${chassis_height}"/>

Commit message: fix(sim): eliminate 10% DiffDrive kinematic error, reduce wheel preload eps to 3mm, and elevate 2D LiDAR above chassis

File: src/amr_sim/urdf/bcr_bot_amr1.xacro (robot description, xacro)
@@ -14,6 +14,6 @@
     <xacro:property name="trolley_wheel_friction" value="0.0"/>
     <xacro:property name="trolley_wheel_radius" value="0.06"/>
-    <!-- a small constant for drive wheel ground engagement -->
-    <xacro:property name="eps" value="0.022"/>
+    <!-- a small constant for drive wheel ground engagement (3mm preload to prevent teeter-totter) -->
+    <xacro:property name="eps" value="0.003"/>
     <xacro:property name="traction_wheel_radius" value="0.1"/>
     <xacro:property name="traction_wheel_width" value="0.05"/>

File: src/amr_sim/urdf/bcr_bot_amr2.xacro (robot description, xacro)
@@ -15,6 +15,6 @@
     <xacro:property name="trolley_wheel_friction" value="0.0"/>
     <xacro:property name="trolley_wheel_radius" value="0.06"/>
-    <!-- a small constant for drive wheel ground engagement -->
-    <xacro:property name="eps" value="0.022"/>
+    <!-- a small constant for drive wheel ground engagement (3mm preload to prevent teeter-totter) -->
+    <xacro:property name="eps" value="0.003"/>
     <xacro:property name="traction_wheel_radius" value="0.1"/>
     <xacro:property name="traction_wheel_width" value="0.05"/>
@@ -118,5 +118,5 @@
             <parent link="base_link"/>
             <child link="two_d_lidar"/>
-            <origin xyz="0.0 0 0.04" rpy="0 0 0" />
+            <origin xyz="0.0 0 0.09" rpy="0 0 0" />
         </joint>
         <gazebo reference="two_d_lidar">

File: src/amr_sim/urdf/gz.xacro (robot description, xacro)
@@ -11,6 +11,6 @@
             <left_joint>middle_left_wheel_joint</left_joint>
             <right_joint>middle_right_wheel_joint</right_joint>
-            <wheel_separation>${traction_track_width+traction_wheel_width-0.01}</wheel_separation>
-            <wheel_radius>${traction_wheel_radius+0.01}</wheel_radius>
+            <wheel_separation>${traction_track_width}</wheel_separation>
+            <wheel_radius>${traction_wheel_radius}</wheel_radius>
             <odom_publish_frequency>30</odom_publish_frequency>
             <max_linear_velocity>1.0</max_linear_velocity>

File: src/amr_sim/urdf/gz_amr2.xacro (robot description, xacro)
@@ -12,12 +12,12 @@
             <left_joint>middle_left_wheel_joint</left_joint>
             <right_joint>middle_right_wheel_joint</right_joint>
-            <wheel_separation>${traction_track_width+traction_wheel_width-0.01}</wheel_separation>
-            <wheel_radius>${traction_wheel_radius+0.01}</wheel_radius>
+            <wheel_separation>${traction_track_width}</wheel_separation>
+            <wheel_radius>${traction_wheel_radius}</wheel_radius>
             <odom_publish_frequency>30</odom_publish_frequency>
             <max_linear_velocity>1.5</max_linear_velocity>
             <max_angular_velocity>1.5</max_angular_velocity>
-            <max_linear_acceleration>3.0</max_linear_acceleration>
-            <max_angular_acceleration>2.5</max_angular_acceleration>
-            <min_linear_acceleration>-2.0</min_linear_acceleration>
+            <max_linear_acceleration>2.5</max_linear_acceleration>
+            <max_angular_acceleration>2.0</max_angular_acceleration>
+            <min_linear_acceleration>-2.5</min_linear_acceleration>
             <topic>/$(arg robot_name)/cmd_vel</topic>
             <odom_topic>/$(arg robot_name)/odom</odom_topic>
